File: PCBs/1S-charging-board_PCB/connectors.kicad_sch (KiCad schematic)
At the start: 2 parts

Commit message: PH20
Parts:
- added PT1: PH2.0, Connector_JST:JST_PH_B2B-PH-K_1x02_P2.00mm_Vertical, symbol Connector_Generic:Conn_01x02
Connections:
- net V+: now also PT1.2 (Pin_2)
- net V-: now also PT1.1 (Pin_1)
Changed lines of the file:
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@@
+	(wire
+		(pts
+			(xy 29.21 74.93) (xy 31.75 74.93)
+		)
+		(stroke
+			(width 0)
+			(type default)
+		)
+	)
 	(wire
 		(pts
@@
 		)
 	)
+	(wire
+		(pts
+			(xy 29.21 72.39) (xy 31.75 72.39)
+		)
+		(stroke
+			(width 0)
+			(type default)
+		)
+	)
 	(label "V-"
 		(at 29.21 49.53 180)
@@
 		)
 	)
+	(label "V-"
+		(at 29.21 74.93 180)
+		(effects
+			(font
+				(size 1.27 1.27)
+			)
+			(justify right bottom)
+		)
+	)
 	(label "V+"
 		(at 29.21 59.69 180)
@@
 	(label "V-"
 		(at 29.21 62.23 180)
+		(effects
+			(font
+				(size 1.27 1.27)
+			)
+			(justify right bottom)
+		)
+	)
+	(label "V+"
+		(at 29.21 72.39 180)
 		(effects
 			(font
@@
 		)
 	)
+	(symbol
+		(lib_id "Connector_Generic:Conn_01x02")
+		(at 36.83 74.93 0)
+		(mirror x)
+		(unit 1)
+		(exclude_from_sim no)
+		(in_bom yes)
+		(on_board yes)
+		(dnp no)
+		(property "Reference" "PT1"
+			(at 36.83 66.04 0)
+			(effects
+				(font
+					(size 1.27 1.27)
+				)
+			)
+		)
+		(property "Value" "PH2.0"
+			(at 36.83 68.58 0)
+			(effects
+				(font
+					(size 1.27 1.27)
+				)
+			)
+		)
+		(property "Footprint" "Connector_JST:JST_PH_B2B-PH-K_1x02_P2.00mm_Vertical"
+			(at 36.83 74.93 0)
+			(effects
+				(font
+					(size 1.27 1.27)
+				)
+				(hide yes)
+			)
+		)
+		(property "Datasheet" "https://www.tme.eu/Document/6eb2005a51a52592b3f19e8a450c54c8/XT30PW-M.pdf"
+			(at 36.83 74.93 0)
+			(effects
+				(font
+					(size 1.27 1.27)
+				)
+				(hide yes)
+			)
+		)
+		(property "Description" "Generic connector, single row, 01x02, script generated (kicad-library-utils/schlib/autogen/connector/)"
+			(at 36.83 74.93 0)
+			(effects
+				(font
+					(size 1.27 1.27)
+				)
+				(hide yes)
+			)
+		)
+		(property "LCSC" "C131337"
+			(at 36.83 74.93 0)
+			(effects
+				(font
+					(size 1.27 1.27)
+				)
+				(hide yes)
+			)
+		)
+		(pin "1"
+		)
+		(pin "2"
+		)
+		(instances
+			(project "1S-charging-board_PCB"
+				(path "/db6a3515-476e-4a92-95a0-11d9c5be923d/28ca4ce6-e862-4878-a716-8a1624d12ea5"
+					(reference "PT5")
+					(unit 1)
+				)
+				(path "/db6a3515-476e-4a92-95a0-11d9c5be923d/64580f3d-940e-4c3c-84c7-7a17efccee74"
+					(reference "PT4")
+					(unit 1)
+				)
+				(path "/db6a3515-476e-4a92-95a0-11d9c5be923d/92ec1954-bd9d-43ac-a983-2031f8a91c06"
+					(reference "PT3")
+					(unit 1)
+				)
+				(path "/db6a3515-476e-4a92-95a0-11d9c5be923d/9311fbfe-8b5e-4b73-befd-ebebffa8f4af"
+					(reference "PT1")
+					(unit 1)
+				)
+				(path "/db6a3515-476e-4a92-95a0-11d9c5be923d/a125f5c8-9d0d-441d-8edb-6650108a9fb8"
+					(reference "PT6")
+					(unit 1)
+				)
+				(path "/db6a3515-476e-4a92-95a0-11d9c5be923d/c15293b2-8fa2-4963-be98-4be6830fbf90"
+					(reference "PT2")
+					(unit 1)
+				)
+			)
+		)
+	)
